File: pcb/avr_apple_remote.brd (EAGLE design)
At the start: 39.7 x 76.2 mm, 18 parts

Commit message: Updated PCB design.
Parts:
- moved LED 1.27 mm to (9.53, 72.4)
Routing:
- net N$10: track 9.72 -> 10.7 mm
Other:
- board text added: "Revision 1.0 March 2015"
Changed lines of the file:
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@@
 <setting verticaltext="up"/>
 </settings>
-<grid distance="0.05" unitdist="inch" unit="inch" style="lines" multiple="1" display="yes" altdistance="0.025" altunitdist="inch" altunit="inch"/>
+<grid distance="1.25" unitdist="mm" unit="mm" style="lines" multiple="1" display="yes" altdistance="0.025" altunitdist="inch" altunit="mm"/>
 <layers>
 <layer number="1" name="Top" color="4" fill="1" visible="yes" active="yes"/>
@@
 <layer number="19" name="Unrouted" color="6" fill="1" visible="yes" active="yes"/>
 <layer number="20" name="Dimension" color="15" fill="1" visible="yes" active="yes"/>
-<layer number="21" name="tPlace" color="7" fill="1" visible="yes" active="yes"/>
+<layer number="21" name="tPlace" color="0" fill="1" visible="yes" active="yes"/>
 <layer number="22" name="bPlace" color="7" fill="1" visible="yes" active="yes"/>
 <layer number="23" name="tOrigins" color="15" fill="1" visible="yes" active="yes"/>
@@
 <wire x1="0" y1="0" x2="39.675" y2="0" width="0" layer="20"/>
 <wire x1="39.675" y1="0" x2="39.675" y2="76.19" width="0" layer="20"/>
-<wire x1="39.675" y1="76.19" x2="0" y2="76.19" width="0" layer="20"/>
 <wire x1="0" y1="76.19" x2="0" y2="0" width="0" layer="20"/>
-<text x="3.175" y="2.54" size="1.778" layer="21" rot="R90">Apple Remote Control</text>
-<text x="38.1" y="2.54" size="1.27" layer="21" rot="R90">Designed by
-Darko, Gabriella &amp; Charlotte Sancanin</text>
+<text x="32.5" y="22.5" size="1.25" layer="21" font="fixed" rot="R270">Designed by
+Darko, Gabriella &amp;
+Charlotte Sancanin</text>
+<text x="28.75" y="3.75" size="1.25" layer="22" font="fixed" rot="MR0">Designed by
+Darko, Gabriella &amp;
+Charlotte Sancanin</text>
+<text x="30" y="21.25" size="1.25" layer="22" font="fixed" rot="MR0">Apple Remote Control</text>
+<text x="3.75" y="5" size="1.25" layer="21" font="fixed" rot="R90">Apple Remote Control</text>
+<text x="25" y="17.5" size="1" layer="22" font="fixed" rot="MR0">Revision 1.0
+March 2015</text>
 </plain>
 <attributes>
@@
 <attribute name="VALUE" x="31.75" y="9.525" size="1.27" layer="27" ratio="10" rot="R270"/>
 </element>
-<element name="SELECT" library="GeekAmmo" package="TAC-SWITCH-PTH" value="" x="19.685" y="45.085"/>
-<element name="IR" library="SparkFun-LED" package="LED5MM" value="" x="19.685" y="72.39"/>
-<element name="RIGHT" library="GeekAmmo" package="TAC-SWITCH-PTH" value="" x="31.115" y="45.085" rot="R180"/>
-<element name="LEFT" library="GeekAmmo" package="TAC-SWITCH-PTH" value="" x="8.255" y="45.085"/>
-<element name="DOWN" library="GeekAmmo" package="TAC-SWITCH-PTH" value="" x="19.685" y="37.465" rot="R180"/>
-<element name="LED" library="SparkFun-LED" package="LED5MM" value="" x="8.255" y="72.39"/>
-<element name="MENU" library="GeekAmmo" package="TAC-SWITCH-PTH" value="" x="19.685" y="29.845" rot="R180"/>
-<element name="IC" library="Atmel_By_element14_Batch_1-00" package="DIP254P762X533-8" value="ATTINY85-20PU" x="23.495" y="67.31" rot="R90">
+<element name="SELECT" library="GeekAmmo" package="TAC-SWITCH-PTH" value="" x="19.685" y="45.085" smashed="yes">
+<attribute name="VALUE" x="17.145" y="40.005" size="1.27" layer="27" ratio="10"/>
+</element>
+<element name="IR" library="SparkFun-LED" package="LED5MM" value="" x="19.685" y="72.39" smashed="yes">
+<attribute name="VALUE" x="22.8854" y="70.5866" size="1.27" layer="27" ratio="10"/>
+</element>
+<element name="RIGHT" library="GeekAmmo" package="TAC-SWITCH-PTH" value="" x="31.115" y="45.085" smashed="yes" rot="R180">
+<attribute name="VALUE" x="33.655" y="50.165" size="1.27" layer="27" ratio="10" rot="R180"/>
+</element>
+<element name="LEFT" library="GeekAmmo" package="TAC-SWITCH-PTH" value="" x="8.255" y="45.085" smashed="yes">
+<attribute name="VALUE" x="5.715" y="40.005" size="1.27" layer="27" ratio="10"/>
+</element>
+<element name="DOWN" library="GeekAmmo" package="TAC-SWITCH-PTH" value="" x="19.685" y="37.465" smashed="yes" rot="R180">
+<attribute name="VALUE" x="22.225" y="42.545" size="1.27" layer="27" ratio="10" rot="R180"/>
+</element>
+<element name="LED" library="SparkFun-LED" package="LED5MM" value="" x="9.525" y="72.39" smashed="yes">
+<attribute name="VALUE" x="12.7254" y="70.5866" size="1.27" layer="27" ratio="10"/>
+</element>
+<element name="MENU" library="GeekAmmo" package="TAC-SWITCH-PTH" value="" x="19.685" y="29.845" smashed="yes" rot="R180">
+<attribute name="VALUE" x="22.225" y="34.925" size="1.27" layer="27" ratio="10" rot="R180"/>
+</element>
+<element name="IC" library="Atmel_By_element14_Batch_1-00" package="DIP254P762X533-8" value="ATTINY85-20PU" x="23.495" y="67.31" smashed="yes" rot="R90">
 <attribute name="PACKAGE" value="PDIP-8" x="23.495" y="67.31" size="1.778" layer="27" rot="R90" display="off"/>
 <attribute name="OC_NEWARK" value="58M3796" x="23.495" y="67.31" size="1.778" layer="27" rot="R90" display="off"/>
@@
 <attribute name="SUPPLIER" value="Atmel" x="23.495" y="67.31" size="1.778" layer="27" rot="R90" display="off"/>
 <attribute name="OC_FARNELL" value="1455162" x="23.495" y="67.31" size="1.778" layer="27" rot="R90" display="off"/>
-</element>
-<element name="UP" library="GeekAmmo" package="TAC-SWITCH-PTH" value="" x="19.685" y="52.705"/>
-<element name="R2" library="rcl" package="0207/10" value="1.8K" x="6.985" y="60.96" rot="R180"/>
-<element name="R3" library="rcl" package="0207/10" value="330" x="6.985" y="57.15" rot="R180"/>
-<element name="R4" library="rcl" package="0207/10" value="680" x="6.985" y="53.34"/>
-<element name="R6" library="rcl" package="0207/10" value="1.8K" x="32.385" y="60.96"/>
-<element name="R7" library="rcl" package="0207/10" value="330" x="32.385" y="57.15"/>
-<element name="R8" library="rcl" package="0207/10" value="680" x="32.385" y="53.34" rot="R180"/>
-<element name="R5" library="rcl" package="0207/10" value="100" x="32.385" y="64.77"/>
-<element name="R1" library="rcl" package="0207/10" value="330" x="6.985" y="64.77"/>
+<attribute name="VALUE" x="12.7" y="60.0456" size="2.0828" layer="27" ratio="10" rot="SR90"/>
+</element>
+<element name="UP" library="GeekAmmo" package="TAC-SWITCH-PTH" value="" x="19.685" y="52.705" smashed="yes">
+<attribute name="VALUE" x="17.145" y="47.625" size="1.27" layer="27" ratio="10"/>
+</element>
+<element name="R2" library="rcl" package="0207/10" value="1.8K" x="6.985" y="60.96" smashed="yes" rot="R180">
+<attribute name="VALUE" x="9.2456" y="61.595" size="1.27" layer="27" ratio="10" rot="R180"/>
+</element>
+<element name="R3" library="rcl" package="0207/10" value="330" x="6.985" y="57.15" smashed="yes" rot="R180">
+<attribute name="VALUE" x="9.2456" y="57.785" size="1.27" layer="27" ratio="10" rot="R180"/>
+</element>
+<element name="R4" library="rcl" package="0207/10" value="680" x="6.985" y="53.34" smashed="yes">
+<attribute name="VALUE" x="4.7244" y="52.705" size="1.27" layer="27" ratio="10"/>
+</element>
+<element name="R6" library="rcl" package="0207/10" value="1.8K" x="32.385" y="60.96" smashed="yes">
+<attribute name="VALUE" x="30.1244" y="60.325" size="1.27" layer="27" ratio="10"/>
+</element>
+<element name="R7" library="rcl" package="0207/10" value="330" x="32.385" y="57.15" smashed="yes">
+<attribute name="VALUE" x="30.1244" y="56.515" size="1.27" layer="27" ratio="10"/>
+</element>
+<element name="R8" library="rcl" package="0207/10" value="680" x="32.385" y="53.34" smashed="yes" rot="R180">
+<attribute name="VALUE" x="34.6456" y="53.975" size="1.27" layer="27" ratio="10" rot="R180"/>
+</element>
+<element name="R5" library="rcl" package="0207/10" value="100" x="32.385" y="64.77" smashed="yes">
+<attribute name="VALUE" x="30.1244" y="64.135" size="1.27" layer="27" ratio="10"/>
+</element>
+<element name="R1" library="rcl" package="0207/10" value="330" x="6.985" y="64.77" smashed="yes">
+<attribute name="VALUE" x="4.7244" y="64.135" size="1.27" layer="27" ratio="10"/>
+</element>
 </elements>
 <signals>
@@
 <polygon width="0.4064" layer="16">
 <vertex x="0" y="76.2"/>
-<vertex x="40.64" y="76.2"/>
-<vertex x="40.64" y="0"/>
+<vertex x="40.005" y="76.2"/>
+<vertex x="40.005" y="0"/>
 <vertex x="0" y="0"/>
 </polygon>
@@
 <contactref element="R6" pad="1"/>
 <contactref element="R2" pad="1"/>
-<wire x1="12.065" y1="60.96" x2="13.97" y2="60.96" width="0.4064" layer="16"/>
-<wire x1="13.97" y1="60.96" x2="15.875" y2="62.865" width="0.4064" layer="16"/>
-<wire x1="15.875" y1="62.865" x2="15.875" y2="66.675" width="0.4064" layer="16"/>
-<wire x1="15.875" y1="66.675" x2="15.24" y2="67.31" width="0.4064" layer="16"/>
 <wire x1="23.495" y1="63.5" x2="19.05" y2="63.5" width="0.4064" layer="16"/>
-<wire x1="19.05" y1="63.5" x2="15.875" y2="66.675" width="0.4064" layer="16"/>
+<wire x1="19.05" y1="63.5" x2="15.24" y2="67.31" width="0.4064" layer="16"/>
 <wire x1="27.305" y1="60.96" x2="26.035" y2="60.96" width="0.4064" layer="16"/>
 <wire x1="26.035" y1="60.96" x2="23.495" y2="63.5" width="0.4064" layer="16"/>
+<wire x1="12.065" y1="60.96" x2="12.7" y2="60.96" width="0.4064" layer="16"/>
+<wire x1="12.7" y1="60.96" x2="15.875" y2="64.135" width="0.4064" layer="16"/>
+<wire x1="15.875" y1="64.135" x2="15.875" y2="67.31" width="0.4064" layer="16"/>
 </signal>
 <signal name="N$11">
@@
 <contactref element="R5" pad="1"/>
 <wire x1="23.495" y1="67.31" x2="23.495" y2="66.675" width="0.4064" layer="1"/>
+<wire x1="25.4" y1="64.77" x2="27.305" y2="64.77" width="0.4064" layer="1"/>
 <wire x1="23.495" y1="66.675" x2="25.4" y2="64.77" width="0.4064" layer="1"/>
-<wire x1="25.4" y1="64.77" x2="27.305" y2="64.77" width="0.4064" layer="1"/>
 </signal>
 <signal name="N$12">
@@
 <contactref element="R1" pad="1"/>
 <wire x1="1.905" y1="64.77" x2="1.905" y2="67.31" width="0.4064" layer="1"/>
-<wire x1="1.905" y1="67.31" x2="6.985" y2="72.39" width="0.4064" layer="1"/>
+<wire x1="1.905" y1="67.31" x2="8.255" y2="72.39" width="0.4064" layer="1"/>
 </signal>
 <signal name="N$7">

Commit message: Updated PCB design with final version - revision 1.0.
Routing:
- net VCC: track 83.7 -> 82.6 mm
- net N$9: track 9.94 -> 10.7 mm
Other:
- board text added: "ATtiny85"
- board text added: "CR2032 BATTERY"
- board text added: "R1"
- board text added: "R2"
- board text added: "R3"
- board text added: "R4"
- board text added: "R5"
- board text added: "R6"
- board text added: "R7"
- board text added: "R8"
Changed lines of the file:
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@@
 <setting verticaltext="up"/>
 </settings>
-<grid distance="1.25" unitdist="mm" unit="mm" style="lines" multiple="1" display="yes" altdistance="0.025" altunitdist="inch" altunit="mm"/>
+<grid distance="0.025" unitdist="inch" unit="inch" style="lines" multiple="1" display="no" altdistance="0.0125" altunitdist="inch" altunit="inch"/>
 <layers>
 <layer number="1" name="Top" color="4" fill="1" visible="yes" active="yes"/>
@@
 <layer number="19" name="Unrouted" color="6" fill="1" visible="yes" active="yes"/>
 <layer number="20" name="Dimension" color="15" fill="1" visible="yes" active="yes"/>
-<layer number="21" name="tPlace" color="0" fill="1" visible="yes" active="yes"/>
+<layer number="21" name="tPlace" color="15" fill="1" visible="yes" active="yes"/>
 <layer number="22" name="bPlace" color="7" fill="1" visible="yes" active="yes"/>
 <layer number="23" name="tOrigins" color="15" fill="1" visible="yes" active="yes"/>
@@
 <wire x1="39.675" y1="0" x2="39.675" y2="76.19" width="0" layer="20"/>
 <wire x1="0" y1="76.19" x2="0" y2="0" width="0" layer="20"/>
-<text x="32.5" y="22.5" size="1.25" layer="21" font="fixed" rot="R270">Designed by
+<text x="32.5" y="23.75" size="1.25" layer="21" font="fixed" rot="R270">Designed by
 Darko, Gabriella &amp;
 Charlotte Sancanin</text>
@@
 <text x="25" y="17.5" size="1" layer="22" font="fixed" rot="MR0">Revision 1.0
 March 2015</text>
+<text x="16.51" y="62.865" size="1" layer="21" font="fixed">ATtiny85</text>
+<text x="17.145" y="12.065" size="1" layer="21" font="fixed">CR2032
+BATTERY</text>
+<text x="7.37" y="64.52" size="0.8" layer="21" font="fixed">R1</text>
+<text x="7.37" y="60.575" size="0.8" layer="21" font="fixed">R2</text>
+<text x="5.195" y="56.9" size="0.8" layer="21" font="fixed">R3</text>
+<text x="5.195" y="53.09" size="0.8" layer="21" font="fixed">R4</text>
+<text x="30.595" y="64.385" size="0.8" layer="21" font="fixed">R5</text>
+<text x="30.595" y="60.575" size="0.8" layer="21" font="fixed">R6</text>
+<text x="32.905" y="56.9" size="0.8" layer="21" font="fixed">R7</text>
+<text x="32.905" y="53.09" size="0.8" layer="21" font="fixed">R8</text>
+<wire x1="0" y1="76.2" x2="39.675" y2="76.2" width="0" layer="20"/>
 </plain>
 <attributes>
@@
 <contactref element="IR" pad="K"/>
 <contactref element="CC" pad="-"/>
-<polygon width="0.4064" layer="16">
-<vertex x="0" y="76.2"/>
-<vertex x="40.005" y="76.2"/>
-<vertex x="40.005" y="0"/>
-<vertex x="0" y="0"/>
-</polygon>
 <contactref element="MENU" pad="3"/>
 <contactref element="DOWN" pad="3"/>
@@
 <contactref element="LEFT" pad="3"/>
 <contactref element="UP" pad="3"/>
+<polygon width="0.4064" layer="16">
+<vertex x="0" y="76.2"/>
+<vertex x="39.6875" y="76.2"/>
+<vertex x="39.6875" y="0"/>
+<vertex x="0" y="0"/>
+</polygon>
 </signal>
 <signal name="N$5">
@@
 <contactref element="IC" pad="8"/>
 <contactref element="CC" pad="+"/>
-<wire x1="15.875" y1="67.31" x2="15.24" y2="67.31" width="0.4064" layer="16"/>
-<wire x1="15.24" y1="67.31" x2="10.16" y2="67.31" width="0.4064" layer="16"/>
+<wire x1="15.875" y1="67.31" x2="10.16" y2="67.31" width="0.4064" layer="16"/>
 <wire x1="10.16" y1="67.31" x2="8.255" y2="65.405" width="0.4064" layer="16"/>
 <wire x1="8.255" y1="65.405" x2="8.255" y2="13.97" width="0.4064" layer="16"/>
@@
 <contactref element="R6" pad="1"/>
 <contactref element="R2" pad="1"/>
-<wire x1="23.495" y1="63.5" x2="19.05" y2="63.5" width="0.4064" layer="16"/>
-<wire x1="19.05" y1="63.5" x2="15.24" y2="67.31" width="0.4064" layer="16"/>
 <wire x1="27.305" y1="60.96" x2="26.035" y2="60.96" width="0.4064" layer="16"/>
 <wire x1="26.035" y1="60.96" x2="23.495" y2="63.5" width="0.4064" layer="16"/>
 <wire x1="12.065" y1="60.96" x2="12.7" y2="60.96" width="0.4064" layer="16"/>
 <wire x1="12.7" y1="60.96" x2="15.875" y2="64.135" width="0.4064" layer="16"/>
-<wire x1="15.875" y1="64.135" x2="15.875" y2="67.31" width="0.4064" layer="16"/>
+<wire x1="15.875" y1="64.135" x2="15.875" y2="66.04" width="0.4064" layer="16"/>
+<wire x1="15.875" y1="66.04" x2="15.875" y2="67.31" width="0.4064" layer="16"/>
+<wire x1="23.495" y1="63.5" x2="18.415" y2="63.5" width="0.4064" layer="16"/>
+<wire x1="18.415" y1="63.5" x2="15.875" y2="66.04" width="0.4064" layer="16"/>
 </signal>
 <signal name="N$11">
@@
 <contactref element="IC" pad="6"/>
 <contactref element="R1" pad="2"/>
-<wire x1="12.065" y1="64.77" x2="18.415" y2="64.77" width="0.4064" layer="1"/>
-<wire x1="18.415" y1="64.77" x2="20.955" y2="67.31" width="0.4064" layer="1"/>
+<wire x1="12.065" y1="64.77" x2="19.685" y2="64.77" width="0.4064" layer="1"/>
+<wire x1="19.685" y1="64.77" x2="20.955" y2="66.04" width="0.4064" layer="1"/>
+<wire x1="20.955" y1="66.04" x2="20.955" y2="67.31" width="0.4064" layer="1"/>
 </signal>
 <signal name="N$10">
